Commit message: feat: add Gazebo-compatible Pro600 official meshes

File: ros2_bridge/ros2_ws/src/mycobot_pro600_description/urdf/pro600_description.urdf.xacro (robot description, xacro)
@@ -3,4 +3,5 @@
   <xacro:arg name="use_ros2_control" default="true"/>
   <xacro:arg name="controllers_file" default=""/>
+  <xacro:arg name="use_gazebo_meshes" default="false"/>
   <xacro:macro name="cylinder_inertia" params="mass radius length">
     <inertial>

File: ros2_bridge/ros2_ws/src/mycobot_pro600_description/urdf/pro600_official_assets.urdf.xacro (robot description, xacro)
@@ -3,9 +3,25 @@
   <xacro:arg name="use_ros2_control" default="true"/>
   <xacro:arg name="controllers_file" default=""/>
+  <xacro:arg name="use_gazebo_meshes" default="false"/>
+  <material name="pro600_dark">
+    <color rgba="0.12 0.14 0.16 1"/>
+  </material>
+  <material name="pro600_white">
+    <color rgba="0.82 0.84 0.86 1"/>
+  </material>
+  <material name="pro600_blue">
+    <color rgba="0.10 0.32 0.58 1"/>
+  </material>
   <link name="base">
     <visual>
       <geometry>
-        <mesh filename="package://mycobot_pro600_description/vendor_ros1/mycobot_description/urdf/mycobot_pro_600/base.dae"/>
-      </geometry>
+        <xacro:if value="$(arg use_gazebo_meshes)">
+          <mesh filename="package://mycobot_pro600_description/meshes/gazebo/base.stl"/>
+        </xacro:if>
+        <xacro:unless value="$(arg use_gazebo_meshes)">
+          <mesh filename="package://mycobot_pro600_description/vendor_ros1/mycobot_description/urdf/mycobot_pro_600/base.dae"/>
+        </xacro:unless>
+      </geometry>
+      <material name="pro600_dark"/>
       <origin xyz="0 0 0" rpy="0 0 0"/>
     </visual>
@@ -25,6 +41,12 @@
     <visual>
       <geometry>
-        <mesh filename="package://mycobot_pro600_description/vendor_ros1/mycobot_description/urdf/mycobot_pro_600/link1.dae"/>
-      </geometry>
+        <xacro:if value="$(arg use_gazebo_meshes)">
+          <mesh filename="package://mycobot_pro600_description/meshes/gazebo/link1.stl"/>
+        </xacro:if>
+        <xacro:unless value="$(arg use_gazebo_meshes)">
+          <mesh filename="package://mycobot_pro600_description/vendor_ros1/mycobot_description/urdf/mycobot_pro_600/link1.dae"/>
+        </xacro:unless>
+      </geometry>
+      <material name="pro600_white"/>
       <origin xyz="0 0 0" rpy="0 0 3.1415926"/>
     </visual>
@@ -44,6 +66,12 @@
     <visual>
       <geometry>
-        <mesh filename="package://mycobot_pro600_description/vendor_ros1/mycobot_description/urdf/mycobot_pro_600/link2.dae"/>
-      </geometry>
+        <xacro:if value="$(arg use_gazebo_meshes)">
+          <mesh filename="package://mycobot_pro600_description/meshes/gazebo/link2.stl"/>
+        </xacro:if>
+        <xacro:unless value="$(arg use_gazebo_meshes)">
+          <mesh filename="package://mycobot_pro600_description/vendor_ros1/mycobot_description/urdf/mycobot_pro_600/link2.dae"/>
+        </xacro:unless>
+      </geometry>
+      <material name="pro600_blue"/>
       <origin xyz="0 0 -0.080" rpy="3.1415926 0 3.1415926"/>
     </visual>
@@ -63,6 +91,12 @@
     <visual>
       <geometry>
-        <mesh filename="package://mycobot_pro600_description/vendor_ros1/mycobot_description/urdf/mycobot_pro_600/link3.dae"/>
-      </geometry>
+        <xacro:if value="$(arg use_gazebo_meshes)">
+          <mesh filename="package://mycobot_pro600_description/meshes/gazebo/link3.stl"/>
+        </xacro:if>
+        <xacro:unless value="$(arg use_gazebo_meshes)">
+          <mesh filename="package://mycobot_pro600_description/vendor_ros1/mycobot_description/urdf/mycobot_pro_600/link3.dae"/>
+        </xacro:unless>
+      </geometry>
+      <material name="pro600_white"/>
       <origin xyz="0 0 -0.0855" rpy="3.1415926 0 3.1415926"/>
     </visual>
@@ -82,6 +116,12 @@
     <visual>
       <geometry>
-        <mesh filename="package://mycobot_pro600_description/vendor_ros1/mycobot_description/urdf/mycobot_pro_600/link4.dae"/>
-      </geometry>
+        <xacro:if value="$(arg use_gazebo_meshes)">
+          <mesh filename="package://mycobot_pro600_description/meshes/gazebo/link4.stl"/>
+        </xacro:if>
+        <xacro:unless value="$(arg use_gazebo_meshes)">
+          <mesh filename="package://mycobot_pro600_description/vendor_ros1/mycobot_description/urdf/mycobot_pro_600/link4.dae"/>
+        </xacro:unless>
+      </geometry>
+      <material name="pro600_blue"/>
       <origin xyz="0 0 0" rpy="0 3.1415926 0"/>
     </visual>
@@ -101,6 +141,12 @@
     <visual>
       <geometry>
-        <mesh filename="package://mycobot_pro600_description/vendor_ros1/mycobot_description/urdf/mycobot_pro_600/link5.dae"/>
-      </geometry>
+        <xacro:if value="$(arg use_gazebo_meshes)">
+          <mesh filename="package://mycobot_pro600_description/meshes/gazebo/link5.stl"/>
+        </xacro:if>
+        <xacro:unless value="$(arg use_gazebo_meshes)">
+          <mesh filename="package://mycobot_pro600_description/vendor_ros1/mycobot_description/urdf/mycobot_pro_600/link5.dae"/>
+        </xacro:unless>
+      </geometry>
+      <material name="pro600_white"/>
       <origin xyz="0 0 0" rpy="0 0 1.5707"/>
     </visual>
@@ -120,9 +166,12 @@
     <visual>
       <geometry>
-        <mesh filename="package://mycobot_pro600_description/vendor_ros1/mycobot_description/urdf/mycobot_pro_600/link6.dae"/>
-      </geometry>
-      <material name="grey">
-        <color rgba="0.5 0.5 0.5 1"/>
-      </material>
+        <xacro:if value="$(arg use_gazebo_meshes)">
+          <mesh filename="package://mycobot_pro600_description/meshes/gazebo/link6.stl"/>
+        </xacro:if>
+        <xacro:unless value="$(arg use_gazebo_meshes)">
+          <mesh filename="package://mycobot_pro600_description/vendor_ros1/mycobot_description/urdf/mycobot_pro_600/link6.dae"/>
+        </xacro:unless>
+      </geometry>
+      <material name="pro600_dark"/>
       <origin xyz="0.03 0 0" rpy="0 -1.5707 0"/>
     </visual>

Commit message: fix: anchor Pro600 base in Gazebo

File: ros2_bridge/ros2_ws/src/mycobot_pro600_description/urdf/pro600_description.urdf.xacro (robot description, xacro)
@@ -4,4 +4,5 @@
   <xacro:arg name="controllers_file" default=""/>
   <xacro:arg name="use_gazebo_meshes" default="false"/>
+  <xacro:arg name="fixed_base" default="true"/>
   <xacro:macro name="cylinder_inertia" params="mass radius length">
     <inertial>
@@ -39,4 +40,12 @@
     <color rgba="0.72 0.74 0.78 1.0"/>
   </material>
+  <xacro:if value="$(arg fixed_base)">
+    <link name="world"/>
+    <joint name="world_to_base" type="fixed">
+      <parent link="world"/>
+      <child link="base_link"/>
+      <origin xyz="0 0 0" rpy="0 0 0"/>
+    </joint>
+  </xacro:if>
   <link name="base_link">
     <visual>

File: ros2_bridge/ros2_ws/src/mycobot_pro600_description/urdf/pro600_official_assets.urdf.xacro (robot description, xacro)
@@ -4,4 +4,5 @@
   <xacro:arg name="controllers_file" default=""/>
   <xacro:arg name="use_gazebo_meshes" default="false"/>
+  <xacro:arg name="fixed_base" default="true"/>
   <material name="pro600_dark">
     <color rgba="0.12 0.14 0.16 1"/>
@@ -13,4 +14,12 @@
     <color rgba="0.10 0.32 0.58 1"/>
   </material>
+  <xacro:if value="$(arg fixed_base)">
+    <link name="world"/>
+    <joint name="world_to_base" type="fixed">
+      <parent link="world"/>
+      <child link="base"/>
+      <origin xyz="0 0 0" rpy="0 0 0"/>
+    </joint>
+  </xacro:if>
   <link name="base">
     <visual>
